Commit message: made basic simulations

File: src/robot_description/urdf/robot_base.urdf.xacro (robot description, xacro)
@@ -21,6 +21,6 @@
     <visual>
       <origin
-        xyz="0 0 0"
-        rpy="1.5707963267949 0 3.14" />
+        xyz="0 0 -.4"
+        rpy="0 0 3.14" />
       <geometry>
         <mesh filename="package://robot_description/meshes/robot_base.stl" />
@@ -34,5 +34,5 @@
     <collision>
       <origin
-        xyz="0 0 0"
+        xyz="0 0 .5"
         rpy="1.5707963267949 0 3.14" />
       <geometry>

File: src/robot_description/urdf/robot_essentials.xacro (robot description, xacro)
@@ -68,5 +68,5 @@
   <joint name="camera_joint" type="fixed">
     <axis xyz="0 1 0" />
-    <origin xyz=".25 0 .25" rpy="0 0 0"/>
+    <origin xyz=".3 0 .45" rpy="0 0 0"/>
     <parent link="base_link"/>
     <child link="camera_link"/>
